File: Hardware/Weather/N81NF-Upgrade/N81NF-Upgrade.sch (KiCad schematic (older format))
At the start: 34 parts, among them P101 CONN_8, P102 CONN_4, P103 CONN_1, P104 CONN_1, P105 CONN_1, U101 A1301, U102 A1301, U103 A1301, U104 A1301, U105 A1301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

Commit message: Basic wind indicator capability
Other:
- note added: "Hall effect sensors are\nA1301KLHLT-T\nFarnell 1791387"
Changed lines of the file:
@@
 Sheet 1 1
 Title ""
-Date "22 jun 2014"
+Date "30 jun 2014"
 Rev ""
 Comp ""
@@
 	7450 1300 7450 1450
 Connection ~ 7450 1450
+Text Notes 3900 2200 0    60   ~ 0
+Hall effect sensors are\nA1301KLHLT-T\nFarnell 1791387
 $EndSCHEMATC
